File: Anthe.brd (EAGLE design)
At the start: 50 x 30 mm, 49 parts, among them J3 POWER_JACK, J4 S3B-XH-A(LF)(SN), P2 S2B-XH-A(LF)(SN), Q3 BSS138, Q4 BSS138, U1 ESP32-C3FH4, U2 WS2812-2020, U4 AP2112K-3.3TRG1, Y2 KYOCERA_INTERNATIONAL_INC._EL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

Commit message: File updates to design
Parts:
- removed ANT1: ANTENNA, adafruit:RN-ANT
- added U$3: PCB_ANTENNA_WIFI, WiFi_PCB_Trace_Antenna:WIFI_ANTENNA
Connections:
- net GND: now also U$3.P$2; no longer ANT1.GND
- net N$2: now also U$3.P$1; no longer ANT1.FEED
Routing:
- net GND: track 9.10 -> 8.29 mm
Changed lines of the file:
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@@
 </autorouter>
 <elements>
-<element name="ANT1" library="adafruit" library_urn="urn:adsk.eagle:library:420" package="RN-ANT" package3d_urn="urn:adsk.eagle:package:6240828/1" value="ANTENNA" x="20.685" y="5.835" smashed="yes" rot="R90"/>
 <element name="C5" library="adafruit" library_urn="urn:adsk.eagle:library:420" package="C0402" package3d_urn="urn:adsk.eagle:package:6240340/1" value="1pF" x="20.64" y="8.525" smashed="yes">
 <attribute name="NAME" x="19.751" y="9.287" size="1.27" layer="25"/>
@@
 <attribute name="VALUE" x="25.59" y="17.418" size="1.27" layer="27"/>
 </element>
+<element name="U$3" library="WiFi_PCB_Trace_Antenna" package="WIFI_ANTENNA" value="PCB_ANTENNA_WIFI" x="20.575" y="5.825" smashed="yes" rot="R180"/>
 </elements>
 <signals>
 <signal name="GND">
-<contactref element="ANT1" pad="GND"/>
 <contactref element="C16" pad="2"/>
 <contactref element="U4" pad="2"/>
@@
 <wire x1="21.29" y1="8.000121875" x2="21" y2="7.3" width="0.8128" layer="1" curve="-45"/>
 <wire x1="21" y1="7.3" x2="20.685" y2="6.539521875" width="0.8128" layer="1" curve="45"/>
-<wire x1="20.685" y1="6.539521875" x2="20.685" y2="4.692" width="0.8128" layer="1"/>
 <contactref element="C12" pad="2"/>
 <via x="18.175" y="20.8" extent="1-16" drill="0.2"/>
@@
 <wire x1="14.821446875" y1="16.725" x2="15.425" y2="16.475" width="0.1524" layer="1" curve="-45"/>
 <wire x1="19.525" y1="16.95" x2="19.5" y2="16.975" width="0.1524" layer="1"/>
+<wire x1="20.65" y1="6.504521875" x2="20.685" y2="6.539521875" width="0.8128" layer="1"/>
+<contactref element="U$3" pad="P$2"/>
+<wire x1="20.575" y1="5.575" x2="20.575" y2="6.273959375" width="0.8128" layer="1"/>
+<wire x1="20.575" y1="6.273959375" x2="20.685" y2="6.539521875" width="0.8128" layer="1" curve="-45"/>
 </signal>
 <signal name="VCC">
@@
 </signal>
 <signal name="N$2">
-<contactref element="ANT1" pad="FEED"/>
 <contactref element="C5" pad="1"/>
 <contactref element="R18" pad="2"/>
@@
 <wire x1="18.325" y1="9.001778125" x2="18.45" y2="8.7" width="0.4064" layer="1" curve="45"/>
 <wire x1="18.45" y1="8.7" x2="18.526" y2="8.51651875" width="0.4064" layer="1" curve="-45"/>
-<wire x1="18.526" y1="5.835" x2="18.526" y2="8.51651875" width="0.4064" layer="1"/>
 <wire x1="18.526" y1="8.51651875" x2="18.546475" y2="8.525" width="0.4064" layer="1" curve="-45"/>
-<wire x1="18.546475" y1="8.525" x2="19.99" y2="8.525" width="0.4064" layer="1"/>
+<wire x1="19.99" y1="8.525" x2="18.546475" y2="8.525" width="0.4064" layer="1"/>
+<wire x1="18.55" y1="8.49251875" x2="18.526" y2="8.51651875" width="0.4064" layer="1"/>
+<contactref element="U$3" pad="P$1"/>
+<wire x1="18.45" y1="8.7" x2="18.475" y2="8.63964375" width="0.4064" layer="1" curve="-45"/>
+<wire x1="18.475" y1="8.63964375" x2="18.475" y2="5.575" width="0.4064" layer="1"/>
 </signal>
 </signals>
