File: Anthe.sch (EAGLE design)
At the start: 49 parts, among them J3 POWER_JACK, J4 S3B-XH-A(LF)(SN), P2 S2B-XH-A(LF)(SN), Q3 BSS138, Q4 BSS138, U1 ESP32-C3FH4, U2 WS2812-2020, U4 AP2112K-3.3TRG1, Y2 KYOCERA_INTERNATIONAL_INC._EL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

Commit message: File updates to design
Parts:
- removed ANT1: ANTENNA, adafruit:ANTENNA
- added U$3: PCB_ANTENNA_WIFI, WiFi_PCB_Trace_Antenna:PCB_ANTENNA_WIFI
Connections:
- net GND: now also U$3.GND; no longer ANT1.GND
- net N$2: now also U$3.FEED; no longer ANT1.FEED
Changed lines of the file:
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@@
 </classes>
 <parts>
-<part name="ANT1" library="adafruit" library_urn="urn:adsk.eagle:library:420" deviceset="ANTENNA" device="" package3d_urn="urn:adsk.eagle:package:6240828/1"/>
 <part name="C5" library="adafruit" library_urn="urn:adsk.eagle:library:420" deviceset="C-US" device="C0402" package3d_urn="urn:adsk.eagle:package:6240340/1" value="1pF"/>
 <part name="GND5" library="supply1" library_urn="urn:adsk.eagle:library:371" deviceset="GND" device=""/>
@@
 <part name="P+10" library="supply1" library_urn="urn:adsk.eagle:library:371" deviceset="VCC" device=""/>
 <part name="FRAME2" library="frames" library_urn="urn:adsk.eagle:library:229" deviceset="DINA4_L" device=""/>
+<part name="U$3" library="WiFi_PCB_Trace_Antenna" deviceset="PCB_ANTENNA_WIFI" device=""/>
 </parts>
 <sheets>
@@
 </plain>
 <instances>
-<instance part="ANT1" gate="G$1" x="891.54" y="154.94" smashed="yes"/>
 <instance part="C5" gate="G$1" x="891.54" y="144.78" smashed="yes">
 <attribute name="NAME" x="892.556" y="145.415" size="1.778" layer="95"/>
@@
 <attribute name="DRAWING_NAME" x="833.12" y="64.77" size="2.54" layer="94"/>
 </instance>
+<instance part="U$3" gate="G$1" x="891.54" y="162.56" smashed="yes"/>
 </instances>
 <busses>
@@
 <net name="GND" class="0">
 <segment>
-<pinref part="ANT1" gate="G$1" pin="GND"/>
-<wire x1="894.08" y1="154.94" x2="894.08" y2="149.86" width="0.1524" layer="91"/>
-<wire x1="894.08" y1="149.86" x2="899.16" y2="149.86" width="0.1524" layer="91"/>
-<wire x1="899.16" y1="149.86" x2="899.16" y2="147.32" width="0.1524" layer="91"/>
+<wire x1="899.16" y1="157.48" x2="899.16" y2="147.32" width="0.1524" layer="91"/>
 <pinref part="GND5" gate="1" pin="GND"/>
+<wire x1="896.62" y1="157.48" x2="899.16" y2="157.48" width="0.1524" layer="91"/>
+<pinref part="U$3" gate="G$1" pin="GND"/>
 </segment>
 <segment>
@@
 <net name="N$2" class="0">
 <segment>
-<pinref part="ANT1" gate="G$1" pin="FEED"/>
 <pinref part="C5" gate="G$1" pin="1"/>
-<wire x1="891.54" y1="154.94" x2="891.54" y2="149.86" width="0.1524" layer="91"/>
+<wire x1="891.54" y1="152.4" x2="891.54" y2="149.86" width="0.1524" layer="91"/>
 <pinref part="R18" gate="G$1" pin="2"/>
 <wire x1="891.54" y1="149.86" x2="891.54" y2="147.32" width="0.1524" layer="91"/>
 <wire x1="889" y1="149.86" x2="891.54" y2="149.86" width="0.1524" layer="91"/>
 <junction x="891.54" y="149.86"/>
-</segment>
-</net>
+<pinref part="U$3" gate="G$1" pin="FEED"/>
+</segment>
+</net>
